Commit message: go2: 切换完整四足仿真并统一定位链路

File: simdog/src/LIO-SAM/config/robot.urdf.xacro (robot description, xacro)
@@ -1,35 +1,5 @@
 <?xml version="1.0"?>
-<robot name="lio" xmlns:xacro="http://tixiaoshan.github.io/">
-  <xacro:property name="PI" value="3.1415926535897931" />
-  <link name="chassis_link"></link>
-  <link name="base_link"></link>
-  <joint name="base_link_joint" type="fixed">
-    <parent link="base_link"/>
-    <child link="chassis_link" />
-    <origin xyz="0 0 0" rpy="0 0 0" />
-  </joint>
-  <link name="lidar_link"> </link>
-  <joint name="lidar_joint" type="fixed">
-    <parent link="base_link" />
-    <child link="lidar_link" />
-    <origin xyz="0 0 0" rpy="0 0 0" />
-  </joint>
-  <link name="imu_link"> </link>
-  <joint name="imu_joint" type="fixed">
-    <parent link="chassis_link" />
-    <child link="imu_link" />
-    <origin xyz="0 0 0" rpy="0 0 0" />
-  </joint>
-  <link name="laser_sensor_frame"> </link>
-  <joint name="laser_joint" type="fixed">
-    <parent link="imu_link" />
-    <child link="laser_sensor_frame" />
-    <origin xyz="0 0 0" rpy="0 0 0" />
-  </joint>
-  <link name="navsat_link"> </link>
-  <joint name="navsat_joint" type="fixed">
-    <parent link="chassis_link" />
-    <child link="navsat_link" />
-    <origin xyz="0 0 0" rpy="0 0 0" />
-  </joint>
+<robot name="go2_lio" xmlns:xacro="http://www.ros.org/wiki/xacro">
+  <!-- LIO-SAM与主仿真共用同一份Go2模型，禁止再定义孤立的lidar_link。 -->
+  <xacro:include filename="$(find go2_description)/xacro/robot_VLP.xacro"/>
 </robot>

File: simdog/src/unitree-go2-ros2/robots/descriptions/go2_description/xacro/velodyne.xacro (robot description, xacro)
@@ -50,5 +50,5 @@
     <gazebo reference="velodyne">
         <sensor name="velodyne-VLP16" type="gpu_ray">
-            <!-- gpu_ray:16×1800=28800条/帧的光线投射交给 GPU(RTX5070),而非拖垮 gzserver 单线程CPU。
+            <!-- gpu_ray:16×1800=28800条/帧的光线投射交给本机RTX 4060 Laptop GPU，而非拖垮gzserver单线程CPU。
                  若换 gpu_ray 后 /velodyne_points 无数据,把这里改回 "ray" 并将下方 samples 降到 512。 -->
             <pose>0 0 0 0 0 0</pose>
